File: esp-walkie-talkie-hw.sch (KiCad schematic (older format))
At the start: 41 parts, among them P1 MIC, P2 PROGRAM, P3 USB_OTG, SW1 SW_VOL+, SW2 SW_VOL-, U1 MCP6004, U2 ESP-12E, U3 XC6210, U4 MCP73831-2-OT

Commit message: Add some hacks to try to reduce the noise
Parts:
- added C? (x2): 10uF, Capacitors_SMD:C_0805, symbol C
- added C?: 100nF, Capacitors_SMD:C_0603, symbol C
- added R?: 1k, Resistors_SMD:R_0603, symbol R
- added R?: 100, Resistors_SMD:R_0603, symbol R
- R3: value 10k -> 1k
- R9: value 1k -> 10k
- U1: value MCP6004 -> LMV324
Connections:
- net +3V3: now also C?.1, C?.1, R?.2; no longer R3.2
- net ADC: now also R?.2; no longer C7.1, R10.2, U1.7
- net GND: now also C?.2, C?.2
- net at C1.1, R1.1, U1.10 (+): now also C?.2
- new net: C7.1, R10.2, R?.1, U1.7
- new net: C?.1, R3.2, R?.1
Changed lines of the file:
@@
 L +3V3 #PWR2
 U 1 1 5AF35ED4
-P 1400 3200
-F 0 "#PWR2" H 1400 3050 50  0001 C CNN
-F 1 "+3V3" H 1400 3340 50  0000 C CNN
-F 2 "" H 1400 3200 50  0000 C CNN
-F 3 "" H 1400 3200 50  0000 C CNN
-	1    1400 3200
+P 1400 2950
+F 0 "#PWR2" H 1400 2800 50  0001 C CNN
+F 1 "+3V3" H 1400 3090 50  0000 C CNN
+F 2 "" H 1400 2950 50  0000 C CNN
+F 3 "" H 1400 2950 50  0000 C CNN
+	1    1400 2950
 	1    0    0    -1
 $EndComp
@@
 P 3250 4150
 F 0 "U1" H 3300 4350 50  0000 C CNN
-F 1 "MCP6004" H 3400 3950 50  0000 C CNN
+F 1 "LMV324" H 3400 3950 50  0000 C CNN
 F 2 "Housings_SOIC:SOIC-14_3.9x8.7mm_Pitch1.27mm" H 3200 4250 50  0001 C CNN
 F 3 "" H 3300 4350 50  0000 C CNN
@@
 P 1400 3450
 F 0 "R3" V 1480 3450 50  0000 C CNN
-F 1 "10k" V 1400 3450 50  0000 C CNN
+F 1 "1k" V 1400 3450 50  0000 C CNN
 F 2 "Resistors_SMD:R_0603" V 1330 3450 50  0001 C CNN
 F 3 "" H 1400 3450 50  0000 C CNN
@@
 	1    0    0    -1
 $EndComp
-Text Label 3900 4150 0    60   ~ 0
+Text Label 4250 4150 0    60   ~ 0
 ADC
 $Comp
@@
 P 4000 5650
 F 0 "U1" H 4050 5850 50  0000 C CNN
-F 1 "MCP6004" H 4150 5450 50  0000 C CNN
+F 1 "LMV324" H 4150 5450 50  0000 C CNN
 F 2 "Housings_SOIC:SOIC-14_3.9x8.7mm_Pitch1.27mm" H 3950 5750 50  0001 C CNN
 F 3 "" H 4050 5850 50  0000 C CNN
@@
 P 4000 6900
 F 0 "U1" H 4050 7100 50  0000 C CNN
-F 1 "MCP6004" H 4150 6700 50  0000 C CNN
+F 1 "LMV324" H 4150 6700 50  0000 C CNN
 F 2 "Housings_SOIC:SOIC-14_3.9x8.7mm_Pitch1.27mm" H 3950 7000 50  0001 C CNN
 F 3 "" H 4050 7100 50  0000 C CNN
@@
 P 2300 6300
 F 0 "U1" H 2350 6500 50  0000 C CNN
-F 1 "MCP6004" H 2450 6100 50  0000 C CNN
+F 1 "LMV324" H 2450 6100 50  0000 C CNN
 F 2 "Housings_SOIC:SOIC-14_3.9x8.7mm_Pitch1.27mm" H 2250 6400 50  0001 C CNN
 F 3 "" H 2350 6500 50  0000 C CNN
@@
 P 2650 5850
 F 0 "R9" V 2730 5850 50  0000 C CNN
-F 1 "1k" V 2650 5850 50  0000 C CNN
+F 1 "10k" V 2650 5850 50  0000 C CNN
 F 2 "Resistors_SMD:R_0603" V 2580 5850 50  0001 C CNN
 F 3 "" H 2650 5850 50  0000 C CNN
@@
 	4200 2150 4300 2150
 Wire Wire Line
-	4300 2150 4300 2350
+	4300 2150 4300 2250
+Wire Wire Line
+	4300 2250 4300 2350
 Wire Wire Line
 	4300 2250 4200 2250
 Wire Wire Line
-	5100 1900 5100 2050
+	5100 1900 5100 1950
+Wire Wire Line
+	5100 1950 5100 2050
 Wire Wire Line
 	5100 1950 5000 1950
@@
 	1950 2250 2400 2250
 Wire Wire Line
-	1950 1650 1950 2250
+	1950 1650 1950 1750
+Wire Wire Line
+	1950 1750 1950 2250
 Wire Wire Line
 	2100 1750 1950 1750
@@
 	2200 1650 2400 1650
 Wire Wire Line
-	1200 4250 1650 4250
+	1200 4250 1400 4250
+Wire Wire Line
+	1400 4250 1650 4250
 Wire Wire Line
 	1400 4250 1400 3900
@@
 Connection ~ 1400 4250
 Wire Wire Line
-	1950 4250 2950 4250
+	1950 4250 2800 4250
+Wire Wire Line
+	2800 4250 2950 4250
 Wire Wire Line
 	3050 4850 2800 4850
 Wire Wire Line
-	2800 4250 2800 5050
+	2800 4250 2800 4850
+Wire Wire Line
+	2800 4850 2800 5050
 Connection ~ 2800 4250
 Wire Wire Line
 	3350 4850 3650 4850
 Wire Wire Line
-	3650 4150 3650 5050
-Wire Wire Line
-	3550 4150 3900 4150
+	3650 4150 3650 4850
+Wire Wire Line
+	3650 4850 3650 5050
+Wire Wire Line
+	3550 4150 3650 4150
 Wire Wire Line
 	3650 5050 3350 5050
@@
 Connection ~ 2800 4850
 Wire Wire Line
-	2250 3600 2750 3600
+	2250 3600 2400 3600
+Wire Wire Line
+	2400 3600 2750 3600
 Wire Wire Line
 	2250 3900 2400 3900
@@
 Connection ~ 3650 4150
 Wire Wire Line
-	1650 5550 3700 5550
-Wire Wire Line
-	900  5550 1350 5550
+	1650 5550 1800 5550
+Wire Wire Line
+	1800 5550 2650 5550
+Wire Wire Line
+	2650 5550 3700 5550
+Wire Wire Line
+	900  5550 1200 5550
+Wire Wire Line
+	1200 5550 1350 5550
 Connection ~ 1800 5550
 Wire Wire Line
 	3700 5750 3500 5750
 Wire Wire Line
-	3500 5750 3500 6350
-Wire Wire Line
-	3500 6200 4550 6200
+	3500 5750 3500 6200
+Wire Wire Line
+	3500 6200 3500 6350
+Wire Wire Line
+	3500 6200 4350 6200
+Wire Wire Line
+	4350 6200 4550 6200
 Wire Wire Line
 	4350 6200 4350 5650
@@
 	3700 7000 3500 7000
 Wire Wire Line
-	3500 6650 3500 7550
+	3500 6650 3500 7000
+Wire Wire Line
+	3500 7000 3500 7550
 Wire Wire Line
 	3500 7550 3750 7550
@@
 	4350 7550 4350 6900
 Wire Wire Line
-	4300 6900 4550 6900
+	4300 6900 4350 6900
+Wire Wire Line
+	4350 6900 4550 6900
 Wire Wire Line
 	1200 5850 1200 6200
@@
 Connection ~ 4350 6900
 Wire Wire Line
+	850  6200 1200 6200
+Wire Wire Line
 	1200 6200 2000 6200
 Wire Wire Line
@@
 	1900 6400 1900 6800
 Wire Wire Line
-	1900 6800 3700 6800
-Wire Wire Line
-	2650 6000 2650 6800
+	1900 6800 2650 6800
+Wire Wire Line
+	2650 6800 3700 6800
+Wire Wire Line
+	2650 6000 2650 6300
+Wire Wire Line
+	2650 6300 2650 6800
 Wire Wire Line
 	2650 6300 2600 6300
@@
 Connection ~ 2650 6800
 Wire Wire Line
-	8400 2100 8400 2350
+	8400 2100 8400 2250
+Wire Wire Line
+	8400 2250 8400 2350
 Wire Wire Line
 	8000 2200 8000 2250
@@
 Connection ~ 8400 2250
 Wire Wire Line
-	7550 1500 8400 1500
+	7550 1500 7850 1500
+Wire Wire Line
+	7850 1500 8400 1500
 Wire Wire Line
 	7150 2100 7150 2200
 Wire Wire Line
-	7150 2200 7650 2200
-Wire Wire Line
-	7650 2200 7650 1800
+	7650 2200 7150 2200
+Wire Wire Line
+	7650 1800 7650 1900
+Wire Wire Line
+	7650 1900 7650 2200
 Wire Wire Line
 	7650 1900 7550 1900
@@
 	9300 2350 9300 2200
 Wire Wire Line
-	9300 1650 9300 1900
+	9300 1650 9300 1700
+Wire Wire Line
+	9300 1700 9300 1900
 Wire Wire Line
 	9300 1700 8800 1700
 Connection ~ 9300 1700
 Wire Wire Line
-	6200 3450 6200 4300
-Wire Wire Line
-	6200 3600 7600 3600
+	6200 3450 6200 3600
+Wire Wire Line
+	6200 3600 6200 4300
+Wire Wire Line
+	6200 3600 6750 3600
+Wire Wire Line
+	6750 3600 7600 3600
 Connection ~ 6200 3600
 Wire Wire Line
 	9100 3800 9100 4550
 Wire Wire Line
-	9400 3450 9400 4250
-Wire Wire Line
-	9100 3600 9900 3600
+	9400 3450 9400 3600
+Wire Wire Line
+	9400 3600 9400 4250
+Wire Wire Line
+	9100 3600 9400 3600
+Wire Wire Line
+	9400 3600 9900 3600
 Connection ~ 9400 3600
 Wire Wire Line
-	6200 4600 6200 4700
-Wire Wire Line
-	6750 4200 6750 4300
-Wire Wire Line
-	6750 4250 6950 4250
+	6200 4600 6200 4650
+Wire Wire Line
+	6200 4650 6200 4700
+Wire Wire Line
+	6750 4200 6750 4250
+Wire Wire Line
+	6750 4250 6750 4300
+Wire Wire Line
+	6750 4250 6900 4250
+Wire Wire Line
+	6900 4250 6950 4250
 Connection ~ 6750 4250
 Wire Wire Line
@@
 Connection ~ 6750 3600
 Wire Wire Line
-	9100 4550 9900 4550
+	9100 4550 9400 4550
+Wire Wire Line
+	9400 4550 9900 4550
 Connection ~ 9400 4550
 Wire Wire Line
@@
 Connection ~ 1400 3600
 Wire Wire Line
-	1400 3300 1400 3200
+	1400 3300 1400 3250
 Wire Wire Line
 	1350 1850 2400 1850
 Wire Wire Line
 	2400 2050 1350 2050
+$Comp
+L C C?
+U 1 1 5B4C9650
+P 1950 3750
+F 0 "C?" H 1975 3850 50  0000 L CNN
+F 1 "10uF" H 1975 3650 50  0000 L CNN
+F 2 "Capacitors_SMD:C_0805" H 1988 3600 50  0001 C CNN
+F 3 "" H 1950 3750 50  0000 C CNN
+	1    1950 3750
+	1    0    0    -1
+$EndComp
+Wire Wire Line
+	1950 3900 1700 3900
+Connection ~ 1700 3900
+Wire Wire Line
+	1950 3600 1950 3250
+Wire Wire Line
+	1950 3250 1400 3250
+$Comp
+L R R?
+U 1 1 5B4C9A70
+P 1400 3100
+F 0 "R?" V 1480 3100 50  0000 C CNN
+F 1 "1k" V 1400 3100 50  0000 C CNN
+F 2 "Resistors_SMD:R_0603" V 1330 3100 50  0001 C CNN
+F 3 "" H 1400 3100 50  0000 C CNN
+	1    1400 3100
+	-1   0    0    1
+$EndComp
+Connection ~ 1400 3250
+$Comp
+L C C?
+U 1 1 5B4C9E7D
+P 850 6050
+F 0 "C?" H 875 6150 50  0000 L CNN
+F 1 "100nF" H 875 5950 50  0000 L CNN
+F 2 "Capacitors_SMD:C_0603" H 888 5900 50  0001 C CNN
+F 3 "" H 850 6050 50  0000 C CNN
+	1    850  6050
+	1    0    0    -1
+$EndComp
+$Comp
+L +3V3 #PWR?
+U 1 1 5B4CA016
+P 850 5900
+F 0 "#PWR?" H 850 5750 50  0001 C CNN
+F 1 "+3V3" H 850 6040 50  0000 C CNN
+F 2 "" H 850 5900 50  0000 C CNN
+F 3 "" H 850 5900 50  0000 C CNN
+	1    850  5900
+	1    0    0    -1
+$EndComp
+$Comp
+L C C?
+U 1 1 5B4CA2B3
+P 1950 2400
+F 0 "C?" H 1975 2500 50  0000 L CNN
+F 1 "10uF" H 1975 2300 50  0000 L CNN
+F 2 "Capacitors_SMD:C_0805" H 1988 2250 50  0001 C CNN
+F 3 "" H 1950 2400 50  0000 C CNN
+	1    1950 2400
+	1    0    0    -1
+$EndComp
+Connection ~ 1950 2250
+$Comp
+L GND #PWR?
+U 1 1 5B4CA38D
+P 1950 2550
+F 0 "#PWR?" H 1950 2300 50  0001 C CNN
+F 1 "GND" H 1950 2400 50  0000 C CNN
+F 2 "" H 1950 2550 50  0000 C CNN
+F 3 "" H 1950 2550 50  0000 C CNN
+	1    1950 2550
+	1    0    0    -1
+$EndComp
+$Comp
+L R R?
+U 1 1 5B4CAF5C
+P 3800 4150
+F 0 "R?" V 3880 4150 50  0000 C CNN
+F 1 "100" V 3800 4150 50  0000 C CNN
+F 2 "Resistors_SMD:R_0603" V 3730 4150 50  0001 C CNN
+F 3 "" H 3800 4150 50  0000 C CNN
+	1    3800 4150
+	0    -1   -1   0
+$EndComp
+Wire Wire Line
+	3950 4150 4250 4150
 $EndSCHEMATC
